File: Project 2a/Maze Schematic.brd (EAGLE design)
At the start: 160 x 100 mm, 14 parts, among them U1 MOD-LED8X8RGB-CONN, U3 POCKETBEAGLE, U6 MOD-LED8X8RGB-CONN

Commit message: Updated Schematic with missing connections
Parts:
- removed U$10, U$7: BUTTON, Buzzer Box:BUTTON-11.5X11.7MM
- added C1, C2, C3: .1uF, Buzzer Box:C0603
- added C4: 10nF, Buzzer Box:C0603
- added R1, R10, R11, R2, R3, R4, R5, R7, R8, R9: 1K, Buzzer Box:R0603
- added R6: 10K, Buzzer Box:R0603
- added SW1, SW2, SW3, SW4, SW5, SW_PWR: BUTTON, Buzzer Box:BUTTON-11.5X11.7MM
- U$1, U$4, U$5, U$6: value BUTTON -> (none); device Buzzer Box:BUTTON-11.5X11.7MM -> Buzzer Box:MOD-LED8X8RGB
- U2: value (none) -> MPU-9250
- moved U$4 193.3 mm to (15.2, 101.6)
- moved U$6 183.5 mm to (76.2, 39.4)
- moved U$5 148.0 mm to (15.2, 39.4)
- moved U$1 128.1 mm to (76.2, 101.6)
- moved U$2 29.5 mm to (19.1, -19.1)
Connections:
- new net BTN1: R1.1, SW1.P$1, SW1.P$2, U3.20
- new net BTN2: R2.1, SW2.P$1, SW2.P$2, U3.55
- new net BTN3: R3.1, SW3.P$1, SW3.P$2, U3.58
- new net BTN4: R4.1, SW4.P$1, SW4.P$2, U3.54
- new net BTN5: R5.1, SW5.P$1, SW5.P$2, U3.60
- new net BUZZER: U$2.+, U3.37
- new net GND: C1.2, C2.2, C3.2, C4.2, SW1.P$3, SW1.P$4, SW2.P$3, SW2.P$4, SW3.P$3, SW3.P$4, SW4.P$3, SW4.P$4, SW5.P$3, SW5.P$4, SW_PWR.P$1, SW_PWR.P$2, U$2.-, U$3.C(-), U$8.C(-), U$9.C(-), U1.5, U1.6, U2.P$18, U2.P$20, U2.P$9, U3.15, U3.16, U3.22, U3.51, U3.57, U6.5, U6.6
- new net I2C2_SCL: R10.1, U2.P$23, U3.28
- new net I2C2_SDA: R11.1, U2.P$24, U3.26
- new net LED-ARRAY1_CS: U3.67, U6.3
- new net LED-ARRAY1_MOSI: U3.12, U6.4
- new net LED-ARRAY1_SCLK: U3.65, U6.2
- new net LED-ARRAY2_CS: U1.3, U3.6
- new net LED-ARRAY2_MOSI: U1.4, U3.61
- new net LED-ARRAY2_SCLK: U1.2, U3.8
- new net LED1: R7.2, U3.44
- new net LED2: R8.2, U3.56
- new net LED3: R9.2, U3.53
- new net MPU_INT: U2.P$12, U3.46
- new net N$1: C2.1, U2.P$10
- new net N$4: C1.1, R6.1, SW_PWR.P$3, SW_PWR.P$4, U3.48
- new net N$5: R7.1, U$9.A(+)
- new net N$6: R8.1, U$8.A(+)
- new net N$7: R9.1, U$3.A(+)
- new net SYS_VDD1_3P3V: R1.2, R2.2, R3.2, R4.2, R5.2
- new net VDD_3P3V: C3.1, C4.1, R10.2, R11.2, U2.P$1, U2.P$13, U2.P$22, U2.P$8, U3.14, U3.59
- new net VDD_5V: U1.1, U3.24, U3.49, U6.1
Routing:
- added copper zone on layer 15, net GND
- added copper zone on layer 2, net VDD_3P3V
Other:
- board size 160 x 100 mm -> 152.4 x 165.1 mm
